File: hdw/HEI_Shift_Light/HEI_Shift_Light/input_power.kicad_sch (KiCad schematic)
At the start: 0 parts

Commit message: Added input power filtering
Parts:
- added C?: (no value), symbol Custom_Library:C_Custom
- added C? (x2): 0.1uF, Capacitors_SMD:C_0603, symbol Custom_Library:C_Custom
- added C?: 100uF, symbol Custom Library:CP_Tant_Custom
- added D?: TVS, Diode_SMD:D_SMB, symbol Custom Library:TVS
- added J?: GND, symbol Connector:Screw_Terminal_01x01
- added J?: VIN, symbol Connector:Screw_Terminal_01x01
- added L?: 10uH, symbol Custom Library:L_Custom
- added R? (x5): R, symbol Custom_Library:R_Custom
- added U1: TPS26624DRCR, Package_SON:VSON-10-1EP_3x3mm_P0.5mm_EP1.65x2.4mm, symbol Custom Library:TPS26624DRCR
Connections:
- new net: D?.1, J?.1 (Pin_1), L?.1
- new net: C?.1, C?.1, L?.2, R?.1, U1.1 (IN)
- new net: R?.1, R?.2, U1.3 (OVP)
- new net: C?.2, R?.2, R?.2, U1.11 (PAD), U1.5 (RTN)
- new net: R?.1, R?.2, U1.2 (UVLO)
- new net: R?.1, U1.7 (ILIM)
- new net: C?.1, U1.8 (DVDT)
- new net +3.3V: R?.1
- new net GND: C?.2, C?.2, C?.2, D?.2, J?.1 (Pin_1), U1.6 (GND)
- new net VIN_PGOOD: R?.2, U1.9 (~{FLT})
- new net Vin: C?.1, U1.10 (OUT)
- no-connect marks 0 -> 1

Commit message: more schematic progress
Parts:
- added R?: R, symbol Custom_Library:R_Custom
Connections:
- net +3.3V is gone; now on net Vin: R?.1
- net GND: now also R?.2
- net VIN_PGOOD: now also R?.1
Other:
- moved on the sheet: R?
Changed lines of the file:
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@@
 	(paper "A")
 	(junction
-		(at 214.63 95.25)
+		(at 224.79 95.25)
 		(diameter 0)
 		(color 0 0 0 0)
@@
 	)
 	(junction
+		(at 224.79 71.12)
+		(diameter 0)
+		(color 0 0 0 0)
+	)
+	(junction
 		(at 240.03 71.12)
 		(diameter 0)
@@
 	(wire
 		(pts
+			(xy 224.79 95.25) (xy 224.79 97.79)
+		)
+		(stroke
+			(width 0)
+			(type default)
+		)
+	)
+	(wire
+		(pts
 			(xy 140.97 71.12) (xy 119.38 71.12)
 		)
@@
 	(wire
 		(pts
+			(xy 198.12 95.25) (xy 224.79 95.25)
+		)
+		(stroke
+			(width 0)
+			(type default)
+		)
+	)
+	(wire
+		(pts
 			(xy 157.48 111.76) (xy 153.67 111.76)
 		)
@@
 	(wire
 		(pts
-			(xy 214.63 95.25) (xy 228.6 95.25)
-		)
-		(stroke
-			(width 0)
-			(type default)
-		)
-	)
-	(wire
-		(pts
-			(xy 214.63 95.25) (xy 214.63 92.71)
+			(xy 224.79 95.25) (xy 238.76 95.25)
+		)
+		(stroke
+			(width 0)
+			(type default)
+		)
+	)
+	(wire
+		(pts
+			(xy 224.79 95.25) (xy 224.79 92.71)
 		)
 		(stroke
@@
 	(wire
 		(pts
+			(xy 224.79 71.12) (xy 240.03 71.12)
+		)
+		(stroke
+			(width 0)
+			(type default)
+		)
+	)
+	(wire
+		(pts
 			(xy 140.97 123.19) (xy 153.67 123.19)
 		)
@@
 	(wire
 		(pts
-			(xy 198.12 95.25) (xy 214.63 95.25)
+			(xy 224.79 71.12) (xy 224.79 85.09)
 		)
 		(stroke
@@
 	(wire
 		(pts
-			(xy 198.12 71.12) (xy 240.03 71.12)
+			(xy 198.12 71.12) (xy 224.79 71.12)
 		)
 		(stroke
@@
 	(global_label "VIN_PGOOD"
 		(shape output)
-		(at 228.6 95.25 0)
+		(at 238.76 95.25 0)
 		(fields_autoplaced yes)
 		(effects
@@
 		)
 		(property "Intersheetrefs" "${INTERSHEET_REFS}"
-			(at 242.0477 95.25 0)
+			(at 252.2077 95.25 0)
 			(hide yes)
 			(show_name no)
@@
 	(symbol
 		(lib_id "Custom_Library:R_Custom")
-		(at 214.63 88.9 0)
+		(at 224.79 88.9 0)
 		(unit 1)
 		(body_style 1)
@@
 		(dnp no)
 		(property "Reference" "R?"
-			(at 212.598 88.9 0)
+			(at 222.758 88.9 0)
 			(show_name no)
 			(do_not_autoplace no)
@@
 		)
 		(property "Value" "R"
-			(at 214.63 88.9 90)
+			(at 224.79 88.9 90)
 			(show_name no)
 			(do_not_autoplace no)
@@
 		)
 		(property "Footprint" ""
-			(at 214.63 88.9 0)
+			(at 224.79 88.9 0)
 			(hide yes)
 			(show_name no)
@@
 		)
 		(property "Datasheet" ""
-			(at 214.63 88.9 0)
+			(at 224.79 88.9 0)
 			(hide yes)
 			(show_name no)
@@
 		)
 		(property "Description" ""
-			(at 214.63 88.9 0)
+			(at 224.79 88.9 0)
 			(show_name no)
 			(do_not_autoplace no)
@@
 		)
 		(property "display_footprint" "0603"
-			(at 217.17 86.868 0)
+			(at 227.33 86.868 0)
 			(show_name no)
 			(do_not_autoplace no)
@@
 		)
 		(property "Tolerance" "1%"
-			(at 217.17 88.9 0)
+			(at 227.33 88.9 0)
 			(show_name no)
 			(do_not_autoplace no)
@@
 		)
 		(property "Wattage" "1/10W"
-			(at 217.424 90.932 0)
+			(at 227.584 90.932 0)
 			(show_name no)
 			(do_not_autoplace no)
@@
 		)
 		(property "Digi-Key PN" ""
-			(at 222.25 78.74 0)
+			(at 232.41 78.74 0)
 			(hide yes)
 			(show_name no)
@@
 	)
 	(symbol
-		(lib_id "power:+3.3V")
-		(at 214.63 85.09 0)
-		(unit 1)
-		(body_style 1)
-		(exclude_from_sim no)
-		(in_bom yes)
-		(on_board yes)
-		(in_pos_files yes)
-		(dnp no)
-		(property "Reference" "#PWR011"
-			(at 214.63 88.9 0)
-			(hide yes)
-			(show_name no)
-			(do_not_autoplace no)
-			(effects
-				(font
-					(size 1.27 1.27)
-				)
-			)
-		)
-		(property "Value" "+3.3V"
-			(at 214.63 81.534 0)
-			(show_name no)
-			(do_not_autoplace no)
-			(effects
-				(font
-					(size 1.27 1.27)
-				)
-			)
-		)
-		(property "Footprint" ""
-			(at 214.63 85.09 0)
-			(hide yes)
-			(show_name no)
-			(do_not_autoplace no)
-			(effects
-				(font
-					(size 1.27 1.27)
-				)
-			)
-		)
-		(property "Datasheet" ""
-			(at 214.63 85.09 0)
-			(hide yes)
-			(show_name no)
-			(do_not_autoplace no)
-			(effects
-				(font
-					(size 1.27 1.27)
-				)
-			)
-		)
-		(property "Description" "Power symbol creates a global label with name \"+3.3V\""
-			(at 214.63 85.09 0)
-			(hide yes)
-			(show_name no)
-			(do_not_autoplace no)
-			(effects
-				(font
-					(size 1.27 1.27)
-				)
-			)
-		)
-		(pin "1"
-		)
-		(instances
-			(project "HEI_Shift_Light"
-				(path "/288c8230-69eb-4ad9-929d-f4630114196f/eeb602ee-2702-41ca-b272-6ee3ac7088d6"
-					(reference "#PWR011")
-					(unit 1)
-				)
-			)
-		)
-	)
-	(symbol
 		(lib_id "Custom_Library:C_Custom")
 		(at 140.97 77.47 0)
@@
 				(path "/288c8230-69eb-4ad9-929d-f4630114196f/eeb602ee-2702-41ca-b272-6ee3ac7088d6"
 					(reference "C?")
+					(unit 1)
+				)
+			)
+		)
+	)
+	(symbol
+		(lib_id "Custom_Library:R_Custom")
+		(at 224.79 101.6 0)
+		(unit 1)
+		(body_style 1)
+		(exclude_from_sim no)
+		(in_bom yes)
+		(on_board yes)
+		(in_pos_files yes)
+		(dnp no)
+		(property "Reference" "R?"
+			(at 222.758 101.6 0)
+			(show_name no)
+			(do_not_autoplace no)
+			(effects
+				(font
+					(size 1.27 1.27)
+				)
+				(justify right)
+			)
+		)
+		(property "Value" "R"
+			(at 224.79 101.6 90)
+			(show_name no)
+			(do_not_autoplace no)
+			(effects
+				(font
+					(size 1.27 1.27)
+				)
+			)
+		)
+		(property "Footprint" ""
+			(at 224.79 101.6 0)
+			(hide yes)
+			(show_name no)
+			(do_not_autoplace no)
+			(effects
+				(font
+					(size 1.27 1.27)
+				)
+			)
+		)
+		(property "Datasheet" ""
+			(at 224.79 101.6 0)
+			(hide yes)
+			(show_name no)
+			(do_not_autoplace no)
+			(effects
+				(font
+					(size 1.27 1.27)
+				)
+			)
+		)
+		(property "Description" ""
+			(at 224.79 101.6 0)
+			(show_name no)
+			(do_not_autoplace no)
+			(effects
+				(font
+					(size 1.27 1.27)
+				)
+			)
+		)
+		(property "display_footprint" "0603"
+			(at 227.33 99.568 0)
+			(show_name no)
+			(do_not_autoplace no)
+			(effects
+				(font
+					(size 1.27 1.27)
+				)
+				(justify left)
+			)
+		)
+		(property "Tolerance" "1%"
+			(at 227.33 101.6 0)
+			(show_name no)
+			(do_not_autoplace no)
+			(effects
+				(font
+					(size 1.27 1.27)
+				)
+				(justify left)
+			)
+		)
+		(property "Wattage" "1/10W"
+			(at 227.584 103.632 0)
+			(show_name no)
+			(do_not_autoplace no)
+			(effects
+				(font
+					(size 1.27 1.27)
+				)
+				(justify left)
+			)
+		)
+		(property "Digi-Key PN" ""
+			(at 232.41 91.44 0)
+			(hide yes)
+			(show_name no)
+			(do_not_autoplace no)
+			(effects
+				(font
+					(size 1.524 1.524)
+				)
+			)
+		)
+		(pin "1"
+		)
+		(pin "2"
+		)
+		(instances
+			(project "HEI_Shift_Light"
+				(path "/288c8230-69eb-4ad9-929d-f4630114196f/eeb602ee-2702-41ca-b272-6ee3ac7088d6"
+					(reference "R?")
 					(unit 1)
 				)
@@
 					(unit 1)
 				)
+			)
+		)
+	)
+	(symbol
+		(lib_id "power:GND")
+		(at 224.79 105.41 0)
+		(unit 1)
+		(body_style 1)
+		(exclude_from_sim no)
+		(in_bom yes)
+		(on_board yes)
+		(in_pos_files yes)
+		(dnp no)
+		(property "Reference" "#PWR011"
+			(at 224.79 111.76 0)
+			(hide yes)
+			(show_name no)
+			(do_not_autoplace no)
+			(effects
+				(font
+					(size 1.27 1.27)
+				)
+			)
+		)
+		(property "Value" "GND"
+			(at 224.79 109.22 0)
+			(show_name no)
+			(do_not_autoplace no)
+			(effects
+				(font
+					(size 1.27 1.27)
+				)
+			)
+		)
+		(property "Footprint" ""
+			(at 224.79 105.41 0)
+			(hide yes)
+			(show_name no)
+			(do_not_autoplace no)
+			(effects
+				(font
+					(size 1.27 1.27)
+				)
+			)
+		)
+		(property "Datasheet" ""
+			(at 224.79 105.41 0)
+			(hide yes)
+			(show_name no)
+			(do_not_autoplace no)
+			(effects
+				(font
+					(size 1.27 1.27)
+				)
+			)
+		)
+		(property "Description" "Power symbol creates a global label with name \"GND\" , ground"
+			(at 224.79 105.41 0)
+			(hide yes)
+			(show_name no)
+			(do_not_autoplace no)
+			(effects
+				(font
+					(size 1.27 1.27)
+				)
+			)
+		)
+		(pin "1"
+		)
+		(instances
+			(project "HEI_Shift_Light"
+				(path "/288c8230-69eb-4ad9-929d-f4630114196f/eeb602ee-2702-41ca-b272-6ee3ac7088d6"
+					(reference "#PWR011")
+					(unit 1)
+				)

Commit message: populated input protection circuit passive components, updated PIC pinout, added stuff to frequency to voltage converter circuit
Parts:
- R?: value R -> 30.1k
- R?: value R -> 15k
- R?: value R -> 100k
- R?: value R -> 42.2k
- R?: value R -> 332k
- R?: value R -> 7.5k
Other:
- note added: "0.88A limit typical"
- note added: "Actual V(UV) rising 10.03 V Error: +0.34% Actual V(OV) rising 15.03 V Error: +0.23% UVLO turn-off (hysteresis) 9.20 V V(UVLOF) = 1.10 V typ OVP reset (hysteresis) 14.03 V"
- note added: "DVDT cap: Min corner: I=2.33 µA, GAIN=23.9 V/V (longest ramp) Typ: I=1.98 µA, GAIN=24.6 V/V Max corner: I=1.68 µA, GAIN=25.2 V/V (shortest ramp - slowest I, widest gain) VOUT target Rise time - min Rise time - typ Rise time - max Slew rate (typ) 10.03 V (UVLO threshold) 18.0 ms 20.6 ms 23.7 ms 0.49 V/ms 12 V (Nominal) 21.5 ms 24.6 ms 28.3 ms 0.49 V/ms 15.03 V (OVP threshold) 27.0 ms 30.9 ms 35.5 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"
- note added: "VIN_PGOOD divider: VEN at VUV (min VOUT) 2.98 V Must be ≥ 0.65 V ✓ VEN at VOV (max VOUT) 4.46 V ✓ Within safe range Divider current at VUV 70.53 µA Keep ≥ 10× EN leakage ✓ V(EN) min = 2.98 V (need ≥ 0.65 V)✓ V(EN) max = 4.46 V✓ Fault: FLT pulls EN to ~0 V (< 0.3 V)"
- moved on the sheet: C?, D?, J?, L?, R?, U1

Commit message: added more shit, RGD LED, LC input filter
Parts:
- removed C?: (no value), symbol Custom_Library:C_Custom
- added C?: 10uF, Capacitors_SMD:C_1206, symbol Custom_Library:C_Custom
- added TP?: VIN, TestPoint:TestPoint_Pad_D1.0mm, symbol Connector:TestPoint
- added TP?: GND, Connector_PinHeader_2.54mm:PinHeader_1x01_P2.54mm_Horizontal, symbol Connector:TestPoint
- C?: footprint (none) -> Capacitor_Tantalum_SMD:CP_EIA-7343-43_Kemet-X; Digi-Key PN (none) -> 399-13127-1-ND; Tolerance Tol -> 20%; Voltage 50V -> 25V; display_footprint Foot -> 7343
- L?: footprint (none) -> Inductor_SMD:L_Vishay_IHLP-2020; Ampacity A -> 2.8A; Digi-Key PN (none) -> 541-IHLP2020CZER100M8ACT-ND; Tolerance Tol -> 20%; display_footprint Foot -> 2020
- renumbered U1 to U?
Connections:
- net GND: now also C?.2, TP?.1
- net Vin: now also C?.1, TP?.1
Other:
- company: (none) -> Drew Maatman
- title: (none) -> HEI Shift Light
