File: hdw/HEI_Shift_Light/HEI_Shift_Light/rgb_led.kicad_sch (KiCad schematic)
At the start: 0 parts

Commit message: added more shit, RGD LED, LC input filter
Parts:
- added D?: Inolux_IN-P55TATRGB, LED_SMD:LED_Avago_PLCC4_3.2x2.8mm_CW, symbol LED:Inolux_IN-P55TATRGB
- added Q? (x3): BSS214NW, Package_TO_SOT_SMD:SOT-323_SC-70, symbol Transistor_FET:BSS214NW
- added R? (x3): 27, Resistors_SMD:R_0603, symbol Custom_Library:R_Custom
- added R? (x3): 10k, Resistors_SMD:R_0603, symbol Custom_Library:R_Custom
- added R? (x2): 91, symbol Custom_Library:R_Custom
- added R?: 150, symbol Custom_Library:R_Custom
Connections:
- new net: Q?.1 (G), R?.1, R?.1 (x3)
- new net: Q?.3 (D), R?.2 (x3)
- new net: D?.1 (KB), R?.1
- new net: D?.2 (KR), R?.1
- new net: D?.3 (KG), R?.1
- new net +5V: D?.4 (AG), D?.5 (AR), D?.6 (AB)
- new net GND: Q?.2 (S), Q?.2 (S), Q?.2 (S), R?.2, R?.2, R?.2
- new net LED_B: R?.2
- new net LED_G: R?.2
- new net LED_R: R?.2
Other:
- note added: "Based on the datasheet, the typical forward current ($I_F$) for testing is 20mA, with an absolute maximum of 25mA. For "maximum brightness" while maintaining reliability, I recommend targeting 20mA. Using Ohm's Law (R = (VCC - VF)*IF with VCC = 5V: +---------+--------+---------------------+-------------------+------------------+ | Channel | Typ Vf | Calculation (20mA) | Recommended Res. | Max Bri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"
- company: (none) -> Drew Maatman
- title: (none) -> HEI Shift Light
