File: hdw/HEI_Shift_Light/USB_UART_Bridge.kicad_sch (KiCad schematic)
At the start: 27 parts, among them U1304 ISO7321C

Commit message: filled in digikey part numbers
Parts:
- C601, C602, C604, C605, C609, C611: renamed from C?; footprint Capacitors_SMD:C_0603 -> Capacitors_SMD:C_0402; Digi-Key PN 1276-1935-1-ND -> 399-7845-1-ND; display_footprint 0603 -> 0402
- C603, C606, C610: renamed from C?; Digi-Key PN 1276-1871-1-ND -> 490-10474-1-ND
- C607, C608: renamed from C?; footprint Capacitors_SMD:C_0603 -> Capacitors_SMD:C_0402; Digi-Key PN 13-CC0603JPNPO9BN470CT-ND -> 311-4037-1-ND; display_footprint 0603 -> 0402
- D601: renamed from D?; Digi-Key PN (none) -> SP0502BAJT-ND
- J601: renamed from J?; Digi-Key PN (none) -> 2073-USB4110-GF-A-1-ND
- L601, L602: renamed from L?; footprint Inductors_SMD:L_0603 -> Inductors_SMD:L_0402; display_footprint (none) -> 0402
- R601, R602, R605, R606: renamed from R?; footprint Resistors_SMD:R_0603 -> Resistors_SMD:R_0402; Digi-Key PN 541-100KHCT-ND -> 541-100KLCT-ND; Wattage 1/10W -> 1/16W; display_footprint 0603 -> 0402
- R603, R604: renamed from R?; footprint Resistors_SMD:R_0603 -> Resistors_SMD:R_0402; Digi-Key PN 541-5306-1-ND -> 541-4082-1-ND; Wattage 1/10W -> 1/16W; display_footprint 0603 -> 0402
- R607, R608: renamed from R?; footprint (none) -> Resistors_SMD:R_0402; Digi-Key PN (none) -> 541-5.10KLCT-ND; Wattage 1/10W -> 1/16W; display_footprint 0603 -> 0402
- gave numbers to parts that had none: 3
- renumbered U1304 to U602

Commit message: fixed a few digikey pns
Parts:
- L601, L602: Digi-Key PN 490-1014-1-ND -> 490-5441-1-ND; MPN (none) -> BLM15AX601SN1D; Manufacturer (none) -> Murata Electronics
Changed lines of the file:
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@@
 			)
 		)
-		(property "Digi-Key PN" "490-1014-1-ND"
+		(property "Digi-Key PN" "490-5441-1-ND"
 			(at 39.624 216.916 0)
 			(hide yes)
@@
 			)
 		)
+    (property "MPN" "BLM15AX601SN1D" (at 247.65 138.43 0)
+      (effects (font (size 1.27 1.27)) (hide yes))
+    )
+    (property "Manufacturer" "Murata Electronics" (at 247.65 138.43 0)
+      (effects (font (size 1.27 1.27)) (hide yes))
+    )
 		(pin "1"
 		)
@@
 			)
 		)
-		(property "Digi-Key PN" "490-1014-1-ND"
+		(property "Digi-Key PN" "490-5441-1-ND"
 			(at 114.046 -150.622 0)
 			(hide yes)
@@
 			)
 		)
+    (property "MPN" "BLM15AX601SN1D" (at 209.55 91.44 0)
+      (effects (font (size 1.27 1.27)) (hide yes))
+    )
+    (property "Manufacturer" "Murata Electronics" (at 209.55 91.44 0)
+      (effects (font (size 1.27 1.27)) (hide yes))
+    )
 		(pin "1"
 		)

Commit message: fixed some digikey pns
Parts:
- C601, C602, C604, C605, C609, C611: Digi-Key PN 399-7845-1-ND -> 1276-7069-1-ND
- C607, C608: Digi-Key PN 311-4037-1-ND -> 311-1021-1-ND
Changed lines of the file:
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@@
 			)
 		)
-		(property "Digi-Key PN" "399-7845-1-ND"
+		(property "Digi-Key PN" "1276-7069-1-ND"
 			(at 103.505 104.14 0)
 			(hide yes)
@@
 			)
 		)
-		(property "Digi-Key PN" "399-7845-1-ND"
+		(property "Digi-Key PN" "1276-7069-1-ND"
 			(at 165.735 40.64 0)
 			(hide yes)
@@
 			)
 		)
-		(property "Digi-Key PN" "399-7845-1-ND"
+		(property "Digi-Key PN" "1276-7069-1-ND"
 			(at 108.585 40.64 0)
 			(hide yes)
@@
 			)
 		)
-		(property "Digi-Key PN" "311-4037-1-ND"
+		(property "Digi-Key PN" "311-1021-1-ND"
 			(at 120.65 116.84 0)
 			(hide yes)
@@
 			)
 		)
-		(property "Digi-Key PN" "311-4037-1-ND"
+		(property "Digi-Key PN" "311-1021-1-ND"
 			(at 142.24 116.84 0)
 			(hide yes)
@@
 			)
 		)
-		(property "Digi-Key PN" "399-7845-1-ND"
+		(property "Digi-Key PN" "1276-7069-1-ND"
 			(at 73.025 67.31 0)
 			(hide yes)
@@
 			)
 		)
-		(property "Digi-Key PN" "399-7845-1-ND"
+		(property "Digi-Key PN" "1276-7069-1-ND"
 			(at 194.945 102.87 0)
 			(hide yes)
@@
 			)
 		)
-		(property "Digi-Key PN" "399-7845-1-ND"
+		(property "Digi-Key PN" "1276-7069-1-ND"
 			(at 55.245 67.31 0)
 			(hide yes)

Commit message: added component datasheet properties
Parts:
- C601, C602, C604, C605, C609, C611: Digi-Key PN 1276-7069-1-ND -> 445-5932-1-ND
Changed lines of the file:
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@@
 			)
 		)
-		(property "Datasheet" ""
+		(property "Datasheet" "https://www.vishay.com/docs/20035/dcrcwe3.pdf"
 			(at 181.61 27.94 0)
 			(hide yes)
@@
 			)
 		)
-		(property "Datasheet" ""
+		(property "Datasheet" "https://pim.murata.com/asset/pim4/ferriteBeadInductortypefilter/ENFA0018_PDF_FERRITEBEADINDUCTORTYPEFILTER"
 			(at 247.65 138.43 0)
 			(hide yes)
@@
 			)
 		)
-		(property "Datasheet" ""
+		(property "Datasheet" "https://www.vishay.com/docs/20035/dcrcwe3.pdf"
 			(at 106.68 109.22 0)
 			(hide yes)
@@
 			)
 		)
-		(property "Datasheet" ""
+		(property "Datasheet" "https://www.vishay.com/docs/20035/dcrcwe3.pdf"
 			(at 106.68 106.68 0)
 			(hide yes)
@@
 			)
 		)
-		(property "Datasheet" ""
+		(property "Datasheet" "https://product.tdk.com/en/system/files/dam/doc/product/capacitor/ceramic/mlcc/charasheet/c1005x7r1h104k050bb.pdf"
 			(at 93.345 114.3 0)
 			(hide yes)
@@
 			)
 		)
-		(property "Digi-Key PN" "1276-7069-1-ND"
+		(property "Digi-Key PN" "445-5932-1-ND"
 			(at 103.505 104.14 0)
 			(hide yes)
@@
 			)
 		)
-		(property "Datasheet" ""
+		(property "Datasheet" "https://pim.murata.com/asset/pim4/ferriteBeadInductortypefilter/ENFA0018_PDF_FERRITEBEADINDUCTORTYPEFILTER"
 			(at 209.55 91.44 0)
 			(hide yes)
@@
 			)
 		)
-		(property "Datasheet" ""
+		(property "Datasheet" "https://search.murata.co.jp/Ceramy/image/img/A01X/G101/ENG/GRM188R61A106KE69-01.pdf"
 			(at 174.625 50.8 0)
 			(hide yes)
@@
 			)
 		)
-		(property "Datasheet" ""
+		(property "Datasheet" "https://product.tdk.com/en/system/files/dam/doc/product/capacitor/ceramic/mlcc/charasheet/c1005x7r1h104k050bb.pdf"
 			(at 155.575 50.8 0)
 			(hide yes)
@@
 			)
 		)
-		(property "Digi-Key PN" "1276-7069-1-ND"
+		(property "Digi-Key PN" "445-5932-1-ND"
 			(at 165.735 40.64 0)
 			(hide yes)
@@
 			)
 		)
-		(property "Datasheet" ""
+		(property "Datasheet" "https://www.vishay.com/docs/20035/dcrcwe3.pdf"
 			(at 194.31 27.94 0)
 			(hide yes)
@@
 			)
 		)
-		(property "Datasheet" ""
+		(property "Datasheet" "https://product.tdk.com/en/system/files/dam/doc/product/capacitor/ceramic/mlcc/charasheet/c1005x7r1h104k050bb.pdf"
 			(at 98.425 50.8 0)
 			(hide yes)
@@
 			)
 		)
-		(property "Digi-Key PN" "1276-7069-1-ND"
+		(property "Digi-Key PN" "445-5932-1-ND"
 			(at 108.585 40.64 0)
 			(hide yes)
@@
 			)
 		)
-		(property "Datasheet" ""
+		(property "Datasheet" "https://www.yageo.com/en/Chart/Download/pdf/CC0402JRNPO9BN470"
 			(at 121.285 114.3 0)
 			(hide yes)
@@
 			)
 		)
-		(property "Datasheet" ""
+		(property "Datasheet" "https://www.vishay.com/docs/20035/dcrcwe3.pdf"
 			(at 73.66 27.94 0)
 			(hide yes)
@@
 			)
 		)
-		(property "Datasheet" ""
+		(property "Datasheet" "https://www.yageo.com/en/Chart/Download/pdf/CC0402JRNPO9BN470"
 			(at 142.875 114.3 0)
 			(hide yes)
@@
 			)
 		)
-		(property "Datasheet" ""
+		(property "Datasheet" "https://www.vishay.com/docs/20035/dcrcwe3.pdf"
 			(at 209.55 115.57 0)
 			(hide yes)
@@
 			)
 		)
-		(property "Datasheet" ""
+		(property "Datasheet" "https://search.murata.co.jp/Ceramy/image/img/A01X/G101/ENG/GRM188R61A106KE69-01.pdf"
 			(at 117.475 50.8 0)
 			(hide yes)
@@
 			)
 		)
-		(property "Datasheet" ""
+		(property "Datasheet" "https://search.murata.co.jp/Ceramy/image/img/A01X/G101/ENG/GRM188R61A106KE69-01.pdf"
 			(at 79.375 77.47 0)
 			(hide yes)
@@
 			)
 		)
-		(property "Datasheet" ""
+		(property "Datasheet" "https://product.tdk.com/en/system/files/dam/doc/product/capacitor/ceramic/mlcc/charasheet/c1005x7r1h104k050bb.pdf"
 			(at 62.865 77.47 0)
 			(hide yes)
@@
 			)
 		)
-		(property "Digi-Key PN" "1276-7069-1-ND"
+		(property "Digi-Key PN" "445-5932-1-ND"
 			(at 73.025 67.31 0)
 			(hide yes)
@@
 			)
 		)
-		(property "Datasheet" ""
+		(property "Datasheet" "https://www.vishay.com/docs/20035/dcrcwe3.pdf"
 			(at 86.36 27.94 0)
 			(hide yes)
@@
 			)
 		)
-		(property "Datasheet" ""
+		(property "Datasheet" "https://www.vishay.com/docs/20035/dcrcwe3.pdf"
 			(at 196.85 115.57 0)
 			(hide yes)
@@
 			)
 		)
-		(property "Datasheet" ""
+		(property "Datasheet" "https://product.tdk.com/en/system/files/dam/doc/product/capacitor/ceramic/mlcc/charasheet/c1005x7r1h104k050bb.pdf"
 			(at 184.785 113.03 0)
 			(hide yes)
@@
 			)
 		)
-		(property "Digi-Key PN" "1276-7069-1-ND"
+		(property "Digi-Key PN" "445-5932-1-ND"
 			(at 194.945 102.87 0)
 			(hide yes)
@@
 			)
 		)
-		(property "Datasheet" ""
+		(property "Datasheet" "https://product.tdk.com/en/system/files/dam/doc/product/capacitor/ceramic/mlcc/charasheet/c1005x7r1h104k050bb.pdf"
 			(at 45.085 77.47 0)
 			(hide yes)
@@
 			)
 		)
-		(property "Digi-Key PN" "1276-7069-1-ND"
+		(property "Digi-Key PN" "445-5932-1-ND"
 			(at 55.245 67.31 0)
 			(hide yes)

Commit message: cleaned up digikey pns
Parts:
- C603, C606, C610: Digi-Key PN 490-10474-1-ND -> 445-C1608X5R1A106K080ACCT-ND
- D601: value SP0502BAJT -> SP0502BAJTG; Digi-Key PN SP0502BAJT-ND -> F3158CT-ND
Changed lines of the file:
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@@
 		(property "Intersheetrefs" "${INTERSHEET_REFS}"
 			(at 227.8772 36.83 0)
-			(hide yes)
 			(show_name no)
 			(do_not_autoplace no)
@@
 		(property "Intersheetrefs" "${INTERSHEET_REFS}"
 			(at 45.4752 36.83 0)
-			(hide yes)
 			(show_name no)
 			(do_not_autoplace no)
@@
 		(property "Intersheetrefs" "${INTERSHEET_REFS}"
 			(at 228.1796 34.29 0)
-			(hide yes)
 			(show_name no)
 			(do_not_autoplace no)
@@
 		(property "Intersheetrefs" "${INTERSHEET_REFS}"
 			(at 45.1728 34.29 0)
-			(hide yes)
 			(show_name no)
 			(do_not_autoplace no)
@@
 		(property "Intersheetrefs" "${INTERSHEET_REFS}"
 			(at 16.9304 101.6 0)
-			(hide yes)
 			(show_name no)
 			(do_not_autoplace no)
@@
 		(property "Intersheetrefs" "${INTERSHEET_REFS}"
 			(at 17.2328 104.14 0)
-			(hide yes)
 			(show_name no)
 			(do_not_autoplace no)
@@
 			)
 		)
-		(property "Value" "SP0502BAJT"
+		(property "Value" "SP0502BAJTG"
 			(at 161.925 116.205 0)
 			(show_name no)
@@
 			)
 		)
-		(property "Digi-Key PN" "SP0502BAJT-ND"
+		(property "Digi-Key PN" "F3158CT-ND"
 			(at 156.21 116.84 0)
 			(hide yes)
@@
 			)
 		)
-		(property "Digi-Key PN" "490-10474-1-ND"
+		(property "Digi-Key PN" "445-C1608X5R1A106K080ACCT-ND"
 			(at 173.99 53.34 0)
 			(hide yes)
@@
 			)
 		)
-		(property "Digi-Key PN" "490-10474-1-ND"
+		(property "Digi-Key PN" "445-C1608X5R1A106K080ACCT-ND"
 			(at 116.84 53.34 0)
 			(hide yes)
@@
 			)
 		)
-		(property "Digi-Key PN" "490-10474-1-ND"
+		(property "Digi-Key PN" "445-C1608X5R1A106K080ACCT-ND"
 			(at 78.74 80.01 0)
 			(hide yes)

Commit message: fixed some footprints, pulled into PCB
Parts:
- DOC601: now left out of the parts list
Changed lines of the file:
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@@
 		(body_style 1)
 		(exclude_from_sim no)
-		(in_bom yes)
-		(on_board yes)
-		(in_pos_files yes)
+		(in_bom no)
+		(on_board no)
+		(in_pos_files no)
 		(dnp no)
 		(property "Reference" "DOC601"
