File: hdw/HEI_Shift_Light/HEI_Shift_Light.kicad_pcb (KiCad board)
At the start: 4 copper layers, 70.7 x 56.9 mm, 111 parts, among them J201 VIN, J401 TACH, J501 PICKIT4, J601 USB_C_Receptacle_USB2.0_16P, Q301 DMN3150LW-7, Q302 DMN3150LW-7, Q701 DMN3150LW-7, Q702 DMN3150LW-7, Q703 DMN3150LW-7, U201 TPS26624DRCR, U301 TPS62153, U401 LM2907, U402 MCP4019-103ELT, U501 PIC18F16Q41, U601 FT234XD, U602 ISO7321C

Commit message: generated gerbers, BOM
Parts:
- added G***: Owl_1_Logo, Custom Footprints Library:Owl_1_Logo, B.Cu at (151.1, 86.7)
Routing:
- added copper zone on F.Cu, net /Input Power/VIN_BATT
Other:
- board text added: "JLCJLCJLCJLC"
